Commit message: changed urdf file

File: urdf/solo12dof_quadruped.urdf (robot description, URDF)
Before this commit: robot solo12dof_quadruped, 8 links, 7 joints
Links:
- added link link_fl_LLM, mass 44.08831168e-3; collision mesh filename=package://solo12_lower_leg_v2_left_side.STL; visual mesh filename=package://solo12_lower_leg_v2_left_side.STL
- added link link_rl_LLM, mass 44.08831168e-3; collision mesh filename=package://solo12_lower_leg_v2_left_side.STL; visual mesh filename=package://solo12_lower_leg_v2_left_side.STL
- added link link_rl_ULM, mass 144.14222037e-3; collision mesh filename=package://solo12_upper_leg_left_side.stl; visual mesh filename=package://solo12_upper_leg_left_side.stl
- added link link_rr_LLM, mass 44.08831168e-3; collision mesh filename=package://solo12_lower_leg_v2_right_side.STL; visual mesh filename=package://solo12_lower_leg_v2_right_side.STL
- added link link_rr_ULM, mass 144.14222037e-3; collision mesh filename=package://solo12_upper_leg_right_side.stl; visual mesh filename=package://solo12_upper_leg_right_side.stl
Joints:
- added joint fl_LLM: type revolute, parent link_fl_ULM, child link_fl_LLM, origin xyz=0 37e-3 -160e-3 rpy=0 0 0, axis 0 1 0, limit lower=-3.141592653589793 upper=3.141592653589793 effort=0 velocity=0
- added joint rl_LLM: type revolute, parent link_rl_ULM, child link_rl_LLM, origin xyz=0 37e-3 -160e-3 rpy=0 0 0, axis 0 1 0, limit lower=-3.141592653589793 upper=3.141592653589793 effort=0 velocity=0
- added joint rl_ULM: type revolute, parent link_rl_hip_fe, child link_rl_ULM, origin xyz=19.65e-3 14e-3 0 rpy=0 0 0, axis 0 1 0, limit lower=-1.5707963267948966 upper=1.5707963267948966 effort=0 velocity=0
- added joint rr_LLM: type revolute, parent link_rr_ULM, child link_rr_LLM, origin xyz=0 -37e-3 -160e-3 rpy=0 0 0, axis 0 1 0, limit lower=-3.141592653589793 upper=3.141592653589793 effort=0 velocity=0
- added joint rr_ULM: type revolute, parent link_rr_hip_fe, child link_rr_ULM, origin xyz=19.65e-3 -14e-3 0 rpy=0 0 0, axis 0 1 0, limit lower=-1.5707963267948966 upper=1.5707963267948966 effort=0 velocity=0
